File: PCB/PCB.kicad_pcb (KiCad board)
At the start: 2 copper layers, 36 parts, among them J1 Screw_Terminal_01x02, J2 Screw_Terminal_01x02, SW1 SW_Push, SW2 SW_Push, U1 MPU-6050, U2 DRV8833PWP, U3 ESP32-S3-MINI-1, U4 AP2112K-3.3

Commit message: PCB Progress
Parts:
- added J3: USB_C_Receptacle_USB2.0_16P, Connector_USB:USB_C_Receptacle_G-Switch_GT-USB-7010ASV, F.Cu at (33.0, 99.1)
- J1: footprint Connector_Phoenix_GMSTB:PhoenixContact_GMSTBA_2,5_2-G_1x02_P7.50mm_Horizontal -> Connector_PinSocket_2.54mm:PinSocket_1x02_P2.54mm_Vertical
- J2: footprint Connector_Phoenix_GMSTB:PhoenixContact_GMSTBA_2,5_2-G_1x02_P7.50mm_Horizontal -> Connector_PinHeader_2.54mm:PinHeader_1x02_P2.54mm_Vertical

Commit message: Finished second PCB
Parts:
- added GND: MountingHole_3.2mm_M3_Pad, MountingHole:MountingHole_3.2mm_M3_Pad, F.Cu at (46.5, 79.0)
- added REF**: MountingHole_3.2mm_M3_Pad, MountingHole:MountingHole_3.2mm_M3_Pad, F.Cu at (46.5, 51.1)
- J3: value USB_C_Receptacle_USB2.0_16P -> USB_C_Receptacle; footprint Connector_USB:USB_C_Receptacle_G-Switch_GT-USB-7010ASV -> Connector_USB:USB_C_Receptacle_Amphenol_12401610E4-2A
- moved R10 78.4 mm to (53.1, 50.2)
- moved D2 78.2 mm to (60.2, 49.7), turned to -90 degrees
- moved R5 73.7 mm to (53.0, 53.6)
- moved R3 68.8 mm to (91.2, 49.7), turned to 90 degrees
- moved R4 68.0 mm to (60.2, 54.3), turned to 90 degrees
- moved R2 59.4 mm to (82.8, 55.0), turned to -90 degrees
- moved C2 54.7 mm to (82.8, 49.7), turned to 90 degrees
- moved C1 53.9 mm to (87.1, 48.9), turned to 180 degrees
- moved R9 53.7 mm to (70.1, 67.7), turned to -90 degrees
- moved R8 53.6 mm to (54.6, 71.0), turned to 90 degrees
- moved R1 52.8 mm to (89.9, 59.8), turned to 90 degrees
- moved R6 52.4 mm to (82.0, 58.8), turned to 180 degrees
- moved C6 50.4 mm to (56.4, 54.3), turned to -90 degrees
- moved R7 49.4 mm to (57.9, 71.0), turned to 90 degrees
- moved J2 47.7 mm to (47.2, 68.3), turned to 180 degrees
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- renumbered SW2 to BOOT, SW1 to RESET
Connections:
- J3 pad A5: Net-(J3-CC1) -> Net-(D1-A)
- R8 pad 1: Net-(J3-CC1) -> Net-(D1-A)
Routing:
- net GND: track 0.00 -> 138.0 mm, vias 0 -> 19
- net BOOT0: track 0.00 -> 87.5 mm, vias 0 -> 2
- net +3.3V: track 0.00 -> 74.0 mm
- net RESET: track 0.00 -> 47.9 mm, vias 0 -> 2
- net SCL: track 0.00 -> 37.1 mm, vias 0 -> 2
- net D-: track 0.00 -> 35.0 mm, vias 0 -> 3
- net D+: track 0.00 -> 33.3 mm, vias 0 -> 3
- net Net-(D1-A): track 0.00 -> 32.5 mm, vias 0 -> 2
- net BIN1: track 0.00 -> 15.0 mm, vias 0 -> 2
- net Net-(U2-AISEN): track 0.00 -> 14.7 mm, vias 0 -> 2
- net AIN1: track 0.00 -> 14.5 mm, vias 0 -> 2
- net SDA: track 0.00 -> 14.4 mm
- net BIN2: track 0.00 -> 14.3 mm, vias 0 -> 2
- net Net-(J3-CC2): track 0.00 -> 12.9 mm, vias 0 -> 2
- net Net-(U2-VINT): track 0.00 -> 12.7 mm, vias 0 -> 2
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- added copper zone on F.Cu, net +3.3V
- added copper zone on F.Cu, net +5V
- added copper zone on B.Cu, net GND
Other:
- board outline added: 51.3 x 43.7 mm
